File: ESP32S3_PlantMonitor/04_ESP32S3_Core.kicad_sch (KiCad schematic)
At the start: 8 parts, among them SW1 SW_Push, SW2 SW_Push, U3 ESP32-S3-WROOM-1

Commit message: Start soil probe input schematic (sheet 06)
Connections:
- no-connect marks 0 -> 31
Changed lines of the file:
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@@
 		(color 0 0 0 0)
+	)
+	(no_connect
+		(at 165.1 104.14)
+	)
+	(no_connect
+		(at 134.62 91.44)
+	)
+	(no_connect
+		(at 134.62 101.6)
+	)
+	(no_connect
+		(at 165.1 86.36)
+	)
+	(no_connect
+		(at 165.1 73.66)
+	)
+	(no_connect
+		(at 134.62 111.76)
+	)
+	(no_connect
+		(at 165.1 88.9)
+	)
+	(no_connect
+		(at 134.62 114.3)
+	)
+	(no_connect
+		(at 134.62 106.68)
+	)
+	(no_connect
+		(at 134.62 83.82)
+	)
+	(no_connect
+		(at 165.1 99.06)
+	)
+	(no_connect
+		(at 165.1 109.22)
+	)
+	(no_connect
+		(at 134.62 99.06)
+	)
+	(no_connect
+		(at 134.62 116.84)
+	)
+	(no_connect
+		(at 165.1 96.52)
+	)
+	(no_connect
+		(at 165.1 93.98)
+	)
+	(no_connect
+		(at 165.1 78.74)
+	)
+	(no_connect
+		(at 134.62 104.14)
+	)
+	(no_connect
+		(at 165.1 101.6)
+	)
+	(no_connect
+		(at 165.1 106.68)
+	)
+	(no_connect
+		(at 165.1 76.2)
+	)
+	(no_connect
+		(at 134.62 96.52)
+	)
+	(no_connect
+		(at 134.62 81.28)
+	)
+	(no_connect
+		(at 165.1 111.76)
+	)
+	(no_connect
+		(at 134.62 93.98)
+	)
+	(no_connect
+		(at 165.1 91.44)
+	)
+	(no_connect
+		(at 165.1 114.3)
+	)
+	(no_connect
+		(at 165.1 71.12)
+	)
+	(no_connect
+		(at 134.62 109.22)
+	)
+	(no_connect
+		(at 165.1 116.84)
+	)
+	(no_connect
+		(at 134.62 78.74)
 	)
 	(wire

Commit message: starting battery schem
Connections:
- net SENS_PWR_EN: now reaches U3.23 (IO21)
- net ADC_SOIL: now reaches U3.39 (IO1)
- no-connect marks 31 -> 29
Changed lines of the file:
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@@
-	)
-	(no_connect
-		(at 165.1 86.36)
 	)
 	(no_connect
@@
 		(at 165.1 116.84)
 	)
-	(no_connect
-		(at 134.62 78.74)
+	(wire
+		(pts
+			(xy 129.54 78.74) (xy 134.62 78.74)
+		)
+		(stroke
+			(width 0)
+			(type default)
+		)
 	)
 	(wire
@@
 		(pts
 			(xy 165.1 81.28) (xy 184.15 81.28)
+		)
+		(stroke
+			(width 0)
+			(type default)
+		)
+	)
+	(wire
+		(pts
+			(xy 165.1 86.36) (xy 177.8 86.36)
 		)
 		(stroke
@@
 			(hide yes)
 			(show_name no)
+			(do_not_autoplace no)
+			(effects
+				(font
+					(size 1.27 1.27)
+				)
+				(justify right)
+			)
+		)
+	)
+	(global_label "SENS_PWR_EN"
+		(shape input)
+		(at 177.8 86.36 270)
+		(fields_autoplaced yes)
+		(effects
+			(font
+				(size 1.27 1.27)
+			)
+			(justify right)
+		)
+		(property "Intersheetrefs" "${INTERSHEET_REFS}"
+			(at 177.8 102.6498 90)
+			(hide yes)
+			(show_name no)
+			(do_not_autoplace no)
+			(effects
+				(font
+					(size 1.27 1.27)
+				)
+				(justify right)
+			)
+		)
+	)
+	(global_label "ADC_SOIL"
+		(shape input)
+		(at 129.54 78.74 180)
+		(fields_autoplaced yes)
+		(effects
+			(font
+				(size 1.27 1.27)
+			)
+			(justify right)
+		)
+		(property "Intersheetrefs" "${INTERSHEET_REFS}"
+			(at 117.7857 78.74 0)
+			(hide yes)
+			(show_name no)
