File: ESP32S3_PlantMonitor/06_Soil_ADC_Input.kicad_sch (KiCad schematic)
At the start: 0 parts

Commit message: starting battery schem
Parts:
- added C14: 100nF, symbol Device:C
- added J2: Conn_01x03, symbol Connector_Generic:Conn_01x03
- added Q1: AO3401A, symbol Transistor_FET:Q_PMOS_GSD
- added R10, R11: 100k, symbol Device:R
Connections:
- new net +3V3: Q1.2 (S), R10.2
- new net ADC_SOIL: C14.2, J2.1 (Pin_1), R11.2
- new net GND: C14.1, J2.3 (Pin_3), R11.1
- new net SENS_PWR_EN: Q1.1 (G), R10.1
- new net SOIL_PWR: J2.2 (Pin_2), Q1.3 (D)
