File: hardware/03_3V3_Power.kicad_sch (KiCad schematic)
At the start: 6 parts, among them U2 AP2112K-3.3

Commit message: Pre-layout finalization and second design review pass (Rev A)
Parts:
- C5: footprint (none) -> Capacitor_SMD:C_0805_2012Metric; LCSC Part (none) -> C15850
- C6, C7: footprint (none) -> Capacitor_SMD:C_0603_1608Metric; LCSC Part (none) -> C15849
- D2: value LED -> LED_YG; footprint (none) -> LED_SMD:LED_0603_1608Metric; LCSC Part (none) -> C2289
- R5: footprint (none) -> Resistor_SMD:R_0603_1608Metric; LCSC Part (none) -> C25804
- U2: LCSC Part (none) -> C51118
Changed lines of the file:
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@@
 			)
 		)
-		(property "Footprint" ""
+		(property "Footprint" "Capacitor_SMD:C_0603_1608Metric"
 			(at 127.9652 100.33 0)
 			(hide yes)
@@
 		)
 		(property "Description" "Unpolarized capacitor"
+			(at 127 96.52 0)
+			(hide yes)
+			(show_name no)
+			(do_not_autoplace no)
+			(effects
+				(font
+					(size 1.27 1.27)
+				)
+			)
+		)
+		(property "LCSC Part" "C15849"
 			(at 127 96.52 0)
 			(hide yes)
@@
 			)
 		)
-		(property "Footprint" ""
+		(property "Footprint" "Capacitor_SMD:C_0805_2012Metric"
 			(at 112.7252 100.33 0)
 			(hide yes)
@@
 		)
 		(property "Description" "Unpolarized capacitor"
+			(at 111.76 96.52 0)
+			(hide yes)
+			(show_name no)
+			(do_not_autoplace no)
+			(effects
+				(font
+					(size 1.27 1.27)
+				)
+			)
+		)
+		(property "LCSC Part" "C15850"
 			(at 111.76 96.52 0)
 			(hide yes)
@@
 			)
 		)
-		(property "Value" "LED"
+		(property "Value" "LED_YG"
 			(at 201.93 110.8074 90)
 			(show_name no)
@@
 			)
 		)
-		(property "Footprint" ""
+		(property "Footprint" "LED_SMD:LED_0603_1608Metric"
 			(at 198.12 107.95 0)
 			(hide yes)
@@
 		(property "Sim.Pins" "1=K 2=A"
 			(at 198.12 107.95 0)
+			(hide yes)
+			(show_name no)
+			(do_not_autoplace no)
+			(effects
+				(font
+					(size 1.27 1.27)
+				)
+			)
+		)
+		(property "LCSC Part" "C2289"
+			(at 198.12 107.95 90)
 			(hide yes)
 			(show_name no)
@@
 			)
 		)
-		(property "Footprint" ""
+		(property "Footprint" "Resistor_SMD:R_0603_1608Metric"
 			(at 196.342 97.79 90)
 			(hide yes)
@@
 		)
 		(property "Description" "Resistor"
+			(at 198.12 97.79 0)
+			(hide yes)
+			(show_name no)
+			(do_not_autoplace no)
+			(effects
+				(font
+					(size 1.27 1.27)
+				)
+			)
+		)
+		(property "LCSC Part" "C25804"
 			(at 198.12 97.79 0)
 			(hide yes)
@@
 			)
 		)
+		(property "LCSC Part" "C51118"
+			(at 149.86 92.71 0)
+			(hide yes)
+			(show_name no)
+			(do_not_autoplace no)
+			(effects
+				(font
+					(size 1.27 1.27)
+				)
+			)
+		)
 		(pin "2"
 		)
@@
 			)
 		)
-		(property "Footprint" ""
+		(property "Footprint" "Capacitor_SMD:C_0603_1608Metric"
 			(at 181.3052 100.33 0)
 			(hide yes)
@@
 			(at 180.34 96.52 0)
 			(hide yes)
+			(show_name no)
+			(do_not_autoplace no)
+			(effects
+				(font
+					(size 1.27 1.27)
+				)
+			)
+		)
+		(property "LCSC Part" "C15849"
+			(at 180.34 96.52 0)
+			(hide yes)

Commit message: pre-order baseline
Other:
- company: (none) -> MuffinByteLabs
- title: (none) -> ESP32-S3 Plant Monitor
Changed lines of the file:
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@@
 	(generator_version "10.0")
 	(paper "A4")
+	(title_block
+		(title "ESP32-S3 Plant Monitor")
+		(date "2026-08-21")
+		(rev "A")
+		(company "MuffinByteLabs")
+		(comment 1 "Designed by Ray Malik")
+		(comment 2 "4-layer JLC04161H-7628, 1.6 mm, HASL lead-free, green mask")
+		(comment 3 "Fabrication and assembly: JLCPCB")
+	)
 	(junction
 		(at 198.12 90.17)
