File: hardware/04_ESP32S3_Core.kicad_sch (KiCad schematic)
At the start: 8 parts, among them SW1 SW_Push, SW2 SW_Push, U3 ESP32-S3-WROOM-1

Commit message: Pre-layout finalization and second design review pass (Rev A)
Parts:
- added TP10, TP9: TestPoint, TestPoint:TestPoint_Pad_D1.5mm, symbol Connector:TestPoint
- added TP11, TP12: TestPoint, TestPoint:TestPoint_THTPad_D2.0mm_Drill1.0mm, symbol Connector:TestPoint
- C10: footprint (none) -> Capacitor_SMD:C_0603_1608Metric; LCSC Part (none) -> C14663
- C8: footprint (none) -> Capacitor_SMD:C_0603_1608Metric; LCSC Part (none) -> C15849
- C9: footprint (none) -> Capacitor_SMD:C_0805_2012Metric; LCSC Part (none) -> C45783
- R6, R7: footprint (none) -> Resistor_SMD:R_0603_1608Metric; LCSC Part (none) -> C25804
- SW1, SW2: footprint (none) -> PlantMonitor_JLC:SW-SMD_4P-L5.1-W5.1-P3.70-LS6.5-TL_H1.5; LCSC Part (none) -> C318884
- U3: LCSC Part (none) -> C2913198
Connections:
- net at R6.1, SW1.1, U3.27 (IO0): now also TP10.1
- net at C8.2, R7.1, SW2.2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: now also TP9.1
- net at U3.36 (RXD0): now also TP12.1
- net at U3.37 (TXD0): now also TP11.1
- no-connect marks 28 -> 26
Other:
- moved on the sheet: R6

Commit message: Component placement: initial floorplan
Connections:
- net GND: now also SW1.1; no longer SW1.2
- net at R6.1, TP10.1, U3.27 (IO0): now also SW1.2; no longer SW1.1
Other:
- moved on the sheet: SW1
Changed lines of the file:
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@@
 	(symbol
 		(lib_id "Switch:SW_Push")
-		(at 106.68 86.36 270)
+		(at 106.68 86.36 90)
 		(unit 1)
 		(body_style 1)
@@
 		(fields_autoplaced yes)
 		(property "Reference" "SW1"
-			(at 110.49 85.0899 90)
+			(at 107.95 85.0899 90)
 			(show_name no)
 			(do_not_autoplace no)
@@
 					(size 1.27 1.27)
 				)
-				(justify left)
+				(justify right)
 			)
 		)
 		(property "Value" "SW_Push"
-			(at 110.49 87.6299 90)
+			(at 107.95 87.6299 90)
 			(show_name no)
 			(do_not_autoplace no)
@@
 					(size 1.27 1.27)
 				)
-				(justify left)
+				(justify right)
 			)
 		)
 		(property "Footprint" "PlantMonitor_JLC:SW-SMD_4P-L5.1-W5.1-P3.70-LS6.5-TL_H1.5"
-			(at 111.76 86.36 0)
+			(at 101.6 86.36 0)
 			(hide yes)
 			(show_name no)
@@
 		)
 		(property "Datasheet" ""
-			(at 111.76 86.36 0)
+			(at 101.6 86.36 0)
 			(hide yes)
 			(show_name no)

Commit message: Routing: bulk of nets complete
Connections:
- net SCL: now also U3.32 (IO39); no longer U3.4 (IO4)
- net SDA: now also U3.31 (IO38); no longer U3.5 (IO5)
- net BOOT: now reaches R6.1, SW1.2, TP10.1, U3.27 (IO0)
- net EN: now reaches C8.2, R7.1, SW2.2, TP9.1, U3.3 (EN)
- net RXD0: now reaches TP12.1, U3.36 (RXD0)
- net TXD0: now reaches TP11.1, U3.37 (TXD0)
Changed lines of the file:
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@@
+	)
+	(no_connect
+		(at 134.62 86.36)
 	)
 	(no_connect
@@
 	)
 	(no_connect
-		(at 165.1 99.06)
-	)
-	(no_connect
 		(at 165.1 109.22)
 	)
@@
 	)
 	(no_connect
+		(at 134.62 88.9)
+	)
+	(no_connect
 		(at 134.62 116.84)
 	)
 	(no_connect
-		(at 165.1 96.52)
-	)
-	(no_connect
 		(at 165.1 93.98)
 	)
@@
 	(wire
 		(pts
-			(xy 121.92 86.36) (xy 121.92 99.06)
-		)
-		(stroke
-			(width 0)
-			(type default)
-		)
-	)
-	(wire
-		(pts
 			(xy 91.44 80.01) (xy 91.44 76.2)
 		)
@@
 	(wire
 		(pts
+			(xy 165.1 99.06) (xy 175.26 99.06)
+		)
+		(stroke
+			(width 0)
+			(type default)
+		)
+	)
+	(wire
+		(pts
 			(xy 73.66 80.01) (xy 91.44 80.01)
 		)
@@
 	(wire
 		(pts
-			(xy 165.1 86.36) (xy 177.8 86.36)
+			(xy 182.88 88.9) (xy 198.12 88.9)
 		)
 		(stroke
@@
 	(wire
 		(pts
-			(xy 129.54 88.9) (xy 134.62 88.9)
-		)
-		(stroke
-			(width 0)
-			(type default)
-		)
-	)
-	(wire
-		(pts
 			(xy 118.11 71.12) (xy 134.62 71.12)
 		)
@@
 	(wire
 		(pts
+			(xy 182.88 86.36) (xy 165.1 86.36)
+		)
+		(stroke
+			(width 0)
+			(type default)
+		)
+	)
+	(wire
+		(pts
+			(xy 165.1 73.66) (xy 200.66 73.66)
+		)
+		(stroke
+			(width 0)
+			(type default)
+		)
+	)
+	(wire
+		(pts
 			(xy 91.44 88.9) (xy 91.44 91.44)
 		)
@@
 	(wire
 		(pts
-			(xy 134.62 86.36) (xy 121.92 86.36)
-		)
-		(stroke
-			(width 0)
-			(type default)
-		)
-	)
-	(wire
-		(pts
 			(xy 123.19 39.37) (xy 123.19 50.8)
 		)
@@
 	(wire
 		(pts
-			(xy 200.66 73.66) (xy 165.1 73.66)
-		)
-		(stroke
-			(width 0)
-			(type default)
-		)
-	)
-	(wire
-		(pts
 			(xy 118.11 54.61) (xy 118.11 50.8)
 		)
@@
 	(wire
 		(pts
+			(xy 165.1 96.52) (xy 175.26 96.52)
+		)
+		(stroke
+			(width 0)
+			(type default)
+		)
+	)
+	(wire
+		(pts
 			(xy 185.42 71.12) (xy 185.42 69.85)
 		)
@@
 	(wire
 		(pts
-			(xy 129.54 99.06) (xy 129.54 88.9)
-		)
-		(stroke
-			(width 0)
-			(type default)
-		)
-	)
-	(wire
-		(pts
 			(xy 95.25 71.12) (xy 105.41 71.12)
 		)
@@
 	(wire
 		(pts
+			(xy 182.88 88.9) (xy 182.88 86.36)
+		)
+		(stroke
+			(width 0)
+			(type default)
+		)
+	)
+	(wire
+		(pts
 			(xy 118.11 50.8) (xy 123.19 50.8)
 		)
@@
 			(width 0)
 			(type default)
+		)
+	)
+	(label "RXD0"
+		(at 193.04 73.66 0)
+		(effects
+			(font
+				(size 1.27 1.27)
+			)
+			(justify left bottom)
+		)
+	)
+	(label "TXD0"
+		(at 177.8 71.12 0)
+		(effects
+			(font
+				(size 1.27 1.27)
+			)
+			(justify left bottom)
+		)
+	)
+	(label "EN"
+		(at 127 71.12 0)
+		(effects
+			(font
+				(size 1.27 1.27)
+			)
+			(justify left bottom)
+		)
+	)
+	(label "BOOT"
+		(at 118.11 76.2 0)
+		(effects
+			(font
+				(size 1.27 1.27)
+			)
+			(justify left bottom)
 		)
 	)
@@
 		)
 	)
-	(global_label "SCL"
-		(shape input)
-		(at 121.92 99.06 270)
-		(fields_autoplaced yes)
-		(effects
-			(font
-				(size 1.27 1.27)
-			)
-			(justify right)
-		)
-		(property "Intersheetrefs" "${INTERSHEET_REFS}"
-			(at 121.92 105.5528 90)
-			(hide yes)
-			(show_name no)
-			(do_not_autoplace no)
-			(effects
-				(font
-					(size 1.27 1.27)
-				)
-				(justify right)
-			)
-		)
-	)
 	(global_label "SENS_PWR_EN"
 		(shape input)
-		(at 177.8 86.36 270)
+		(at 198.12 88.9 270)
 		(fields_autoplaced yes)
 		(effects
@@
 		)
 		(property "Intersheetrefs" "${INTERSHEET_REFS}"
-			(at 177.8 102.6498 90)
+			(at 198.12 105.1898 90)
 			(hide yes)
 			(show_name no)
@@
 		)
 	)
-	(global_label "SDA"
+	(global_label "SCL"
 		(shape input)
-		(at 129.54 99.06 270)
+		(at 175.26 99.06 270)
 		(fields_autoplaced yes)
 		(effects
@@
 		)
 		(property "Intersheetrefs" "${INTERSHEET_REFS}"
-			(at 129.54 105.6133 90)
+			(at 175.26 105.5528 90)
 			(hide yes)
 			(show_name no)
@@
 			)
 		)
+	)
+	(global_label "SDA"
+		(shape input)
+		(at 175.26 96.52 90)
+		(fields_autoplaced yes)
+		(effects
+			(font
+				(size 1.27 1.27)
+			)
+			(justify left)
+		)
+		(property "Intersheetrefs" "${INTERSHEET_REFS}"
+			(at 175.26 89.9667 90)
+			(hide yes)
+			(show_name no)
+			(do_not_autoplace no)
+			(effects
+				(font
+					(size 1.27 1.27)
+				)
+				(justify left)
+			)
+		)

Commit message: pre-order baseline
Other:
- company: (none) -> MuffinByteLabs
- title: (none) -> ESP32-S3 Plant Monitor
Changed lines of the file:
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@@
 	(generator_version "10.0")
 	(paper "A4")
+	(title_block
+		(title "ESP32-S3 Plant Monitor")
+		(date "2026-08-21")
+		(rev "A")
+		(company "MuffinByteLabs")
+		(comment 1 "Designed by Ray Malik")
+		(comment 2 "4-layer JLC04161H-7628, 1.6 mm, HASL lead-free, green mask")
+		(comment 3 "Fabrication and assembly: JLCPCB")
+	)
 	(junction
 		(at 149.86 57.15)
