File: hardware/05_I2C_Sensors.kicad_sch (KiCad schematic)
At the start: 7 parts, among them U4 BME280, U5 VEML7700-TT

Commit message: Pre-layout finalization and second design review pass (Rev A)
Parts:
- C11, C12, C13: footprint (none) -> Capacitor_SMD:C_0603_1608Metric; LCSC Part (none) -> C14663
- R8, R9: footprint (none) -> Resistor_SMD:R_0603_1608Metric; LCSC Part (none) -> C23162
- U4: LCSC Part (none) -> C92489
Changed lines of the file:
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@@
 			)
 		)
-		(property "Footprint" ""
+		(property "Footprint" "Resistor_SMD:R_0603_1608Metric"
 			(at 199.39 108.458 90)
 			(hide yes)
@@
 		(property "Description" "Resistor"
 			(at 199.39 106.68 0)
+			(hide yes)
+			(show_name no)
+			(do_not_autoplace no)
+			(effects
+				(font
+					(size 1.27 1.27)
+				)
+			)
+		)
+		(property "LCSC Part" "C23162"
+			(at 199.39 106.68 90)
 			(hide yes)
 			(show_name no)
@@
 			)
 		)
-		(property "Footprint" ""
+		(property "Footprint" "Capacitor_SMD:C_0603_1608Metric"
 			(at 105.41 77.7748 0)
 			(hide yes)
@@
 		(property "Description" "Unpolarized capacitor"
 			(at 101.6 78.74 0)
+			(hide yes)
+			(show_name no)
+			(do_not_autoplace no)
+			(effects
+				(font
+					(size 1.27 1.27)
+				)
+			)
+		)
+		(property "LCSC Part" "C14663"
+			(at 101.6 78.74 90)
 			(hide yes)
 			(show_name no)
@@
 			)
 		)
+		(property "LCSC Part" "C92489"
+			(at 120.65 95.25 0)
+			(hide yes)
+			(show_name no)
+			(do_not_autoplace no)
+			(effects
+				(font
+					(size 1.27 1.27)
+				)
+			)
+		)
 		(pin "2"
 		)
@@
 			)
 		)
-		(property "Footprint" ""
+		(property "Footprint" "Capacitor_SMD:C_0603_1608Metric"
 			(at 180.0352 91.44 0)
 			(hide yes)
@@
 		)
 		(property "Description" "Unpolarized capacitor"
+			(at 179.07 87.63 0)
+			(hide yes)
+			(show_name no)
+			(do_not_autoplace no)
+			(effects
+				(font
+					(size 1.27 1.27)
+				)
+			)
+		)
+		(property "LCSC Part" "C14663"
 			(at 179.07 87.63 0)
 			(hide yes)
@@
 			)
 		)
-		(property "Footprint" ""
+		(property "Footprint" "Resistor_SMD:R_0603_1608Metric"
 			(at 199.39 78.232 90)
 			(hide yes)
@@
 		(property "Description" "Resistor"
 			(at 199.39 80.01 0)
+			(hide yes)
+			(show_name no)
+			(do_not_autoplace no)
+			(effects
+				(font
+					(size 1.27 1.27)
+				)
+			)
+		)
+		(property "LCSC Part" "C23162"
+			(at 199.39 80.01 90)
 			(hide yes)
 			(show_name no)
@@
 			)
 		)
-		(property "Footprint" ""
+		(property "Footprint" "Capacitor_SMD:C_0603_1608Metric"
 			(at 134.62 79.7052 0)
 			(hide yes)
@@
 			(hide yes)
 			(show_name no)
+			(do_not_autoplace no)
+			(effects
+				(font
+					(size 1.27 1.27)
+				)
+			)
+		)
+		(property "LCSC Part" "C14663"
+			(at 138.43 78.74 90)
+			(hide yes)
+			(show_name no)

Commit message: pre-order baseline
Other:
- company: (none) -> MuffinByteLabs
- title: (none) -> ESP32-S3 Plant Monitor
Changed lines of the file:
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@@
 	(generator_version "10.0")
 	(paper "A4")
+	(title_block
+		(title "ESP32-S3 Plant Monitor")
+		(date "2026-08-21")
+		(rev "A")
+		(company "MuffinByteLabs")
+		(comment 1 "Designed by Ray Malik")
+		(comment 2 "4-layer JLC04161H-7628, 1.6 mm, HASL lead-free, green mask")
+		(comment 3 "Fabrication and assembly: JLCPCB")
+	)
 	(junction
 		(at 120.65 116.84)
