File: hardware/07_Battery_Charger.kicad_sch (KiCad schematic)
At the start: 15 parts, among them J3 Conn_01x02, Q2 AO3401A, Q3 AO3401A, U6 MCP73831-2-OT

Commit message: Pre-layout finalization and second design review pass (Rev A)
Parts:
- C15, C16: value 4.7u -> 4.7uF; footprint (none) -> Capacitor_SMD:C_0603_1608Metric; LCSC Part (none) -> C19666
- C17: footprint (none) -> Capacitor_SMD:C_0603_1608Metric; LCSC Part (none) -> C14663
- C18: value 1u -> 1uF; footprint (none) -> Capacitor_SMD:C_0603_1608Metric; LCSC Part (none) -> C15849
- D3: value LED -> LED_RED; footprint (none) -> LED_SMD:LED_0603_1608Metric; LCSC Part (none) -> C2286
- D4: LCSC Part (none) -> C2480
- J3: footprint (none) -> Connector_JST:JST_PH_S2B-PH-K_1x02_P2.00mm_Horizontal; LCSC Part (none) -> C173752
- Q2, Q3: footprint (none) -> Package_TO_SOT_SMD:SOT-23; LCSC Part (none) -> C15127
- R12: footprint (none) -> Resistor_SMD:R_0603_1608Metric; LCSC Part (none) -> C23179
- R13, R16: footprint (none) -> Resistor_SMD:R_0603_1608Metric; LCSC Part (none) -> C25804
- R14, R15: footprint (none) -> Resistor_SMD:R_0603_1608Metric; LCSC Part (none) -> C25803
- U6: LCSC Part (none) -> C424093
Changed lines of the file:
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@@
 		)
 	)
-	(label "VBAT"
-		(at 179.07 87.63 0)
+	(global_label "VBAT"
+		(shape input)
+		(at 179.07 87.63 90)
+		(fields_autoplaced yes)
 		(effects
 			(font
 				(size 1.27 1.27)
 			)
-			(justify left bottom)
+			(justify left)
+		)
+		(property "Intersheetrefs" "${INTERSHEET_REFS}"
+			(at 179.07 80.23 90)
+			(hide yes)
+			(show_name no)
+			(do_not_autoplace no)
+			(effects
+				(font
+					(size 1.27 1.27)
+				)
+				(justify left)
+			)
 		)
 	)
@@
 			)
 		)
-		(property "Footprint" ""
+		(property "Footprint" "Resistor_SMD:R_0603_1608Metric"
 			(at 231.902 78.74 90)
 			(hide yes)
@@
 			)
 		)
+		(property "LCSC Part" "C25804"
+			(at 233.68 78.74 0)
+			(hide yes)
+			(show_name no)
+			(do_not_autoplace no)
+			(effects
+				(font
+					(size 1.27 1.27)
+				)
+			)
+		)
 		(pin "1"
 		)
@@
 			)
 		)
-		(property "Footprint" ""
+		(property "Footprint" "Resistor_SMD:R_0603_1608Metric"
 			(at 168.402 95.25 90)
 			(hide yes)
@@
 			)
 		)
+		(property "LCSC Part" "C25803"
+			(at 170.18 95.25 0)
+			(hide yes)
+			(show_name no)
+			(do_not_autoplace no)
+			(effects
+				(font
+					(size 1.27 1.27)
+				)
+			)
+		)
 		(pin "1"
 		)
@@
 			)
 		)
-		(property "Value" "4.7u"
+		(property "Value" "4.7uF"
 			(at 158.75 104.14 0)
 			(show_name no)
@@
 			)
 		)
-		(property "Footprint" ""
+		(property "Footprint" "Capacitor_SMD:C_0603_1608Metric"
 			(at 164.7952 102.87 0)
 			(hide yes)
@@
 		)
 		(property "Description" "Unpolarized capacitor"
+			(at 163.83 99.06 0)
+			(hide yes)
+			(show_name no)
+			(do_not_autoplace no)
+			(effects
+				(font
+					(size 1.27 1.27)
+				)
+			)
+		)
+		(property "LCSC Part" "C19666"
 			(at 163.83 99.06 0)
 			(hide yes)
@@
 			)
 		)
-		(property "Footprint" ""
+		(property "Footprint" "Package_TO_SOT_SMD:SOT-23"
 			(at 204.47 90.17 0)
 			(hide yes)
@@
 			)
 		)
+		(property "LCSC Part" "C15127"
+			(at 207.01 85.09 90)
+			(hide yes)
+			(show_name no)
+			(do_not_autoplace no)
+			(effects
+				(font
+					(size 1.27 1.27)
+				)
+			)
+		)
 		(pin "3"
 		)
@@
 			)
 		)
-		(property "Footprint" ""
+		(property "Footprint" "Capacitor_SMD:C_0603_1608Metric"
 			(at 183.8452 128.27 0)
 			(hide yes)
@@
 			)
 		)
+		(property "LCSC Part" "C14663"
+			(at 182.88 124.46 0)
+			(hide yes)
+			(show_name no)
+			(do_not_autoplace no)
+			(effects
+				(font
+					(size 1.27 1.27)
+				)
+			)
+		)
 		(pin "1"
 		)
@@
 			)
 		)
-		(property "Footprint" ""
+		(property "Footprint" "Package_TO_SOT_SMD:SOT-23"
 			(at 191.77 111.76 0)
 			(hide yes)
@@
 			)
 		)
+		(property "LCSC Part" "C15127"
+			(at 196.85 109.22 90)
+			(hide yes)
+			(show_name no)
+			(do_not_autoplace no)
+			(effects
+				(font
+					(size 1.27 1.27)
+				)
+			)
+		)
 		(pin "3"
 		)
@@
 			)
 		)
-		(property "Value" "LED"
+		(property "Value" "LED_RED"
 			(at 100.33 108.2674 90)
 			(show_name no)
@@
 			)
 		)
-		(property "Footprint" ""
+		(property "Footprint" "LED_SMD:LED_0603_1608Metric"
 			(at 96.52 105.41 0)
 			(hide yes)
@@
 			)
 		)
+		(property "LCSC Part" "C2286"
+			(at 96.52 105.41 90)
+			(hide yes)
+			(show_name no)
+			(do_not_autoplace no)
+			(effects
+				(font
+					(size 1.27 1.27)
+				)
+			)
+		)
 		(pin "1"
 		)
@@
 			)
 		)
-		(property "Footprint" ""
+		(property "Footprint" "Connector_JST:JST_PH_S2B-PH-K_1x02_P2.00mm_Horizontal"
 			(at 200.66 133.35 0)
 			(hide yes)
@@
 			)
 		)
+		(property "LCSC Part" "C173752"
+			(at 200.66 133.35 0)
+			(hide yes)
+			(show_name no)
+			(do_not_autoplace no)
+			(effects
+				(font
+					(size 1.27 1.27)
+				)
+			)
+		)
 		(pin "2"
 		)
@@
 			)
 		)
-		(property "Footprint" ""
+		(property "Footprint" "Resistor_SMD:R_0603_1608Metric"
 			(at 168.402 113.03 90)
 			(hide yes)
@@
 			)
 		)
+		(property "LCSC Part" "C25803"
+			(at 170.18 113.03 0)
+			(hide yes)
+			(show_name no)
+			(do_not_autoplace no)
+			(effects
+				(font
+					(size 1.27 1.27)
+				)
+			)
+		)
 		(pin "1"
 		)
@@
 			)
 		)
-		(property "Footprint" ""
+		(property "Footprint" "Resistor_SMD:R_0603_1608Metric"
 			(at 94.742 96.52 90)
 			(hide yes)
@@
 			)
 		)
+		(property "LCSC Part" "C23179"
+			(at 96.52 96.52 0)
+			(hide yes)
+			(show_name no)
+			(do_not_autoplace no)
+			(effects
+				(font
+					(size 1.27 1.27)
+				)
+			)
+		)
 		(pin "1"
 		)
@@
 			)
 		)
+		(property "LCSC Part" "C2480"
+			(at 215.9 76.2 90)
+			(hide yes)
+			(show_name no)
+			(do_not_autoplace no)
+			(effects
+				(font
+					(size 1.27 1.27)
+				)
+			)
+		)
 		(pin "2"
 		)
@@
 			)
 		)
+		(property "LCSC Part" "C424093"
+			(at 128.27 90.17 0)
+			(hide yes)
+			(show_name no)
+			(do_not_autoplace no)
+			(effects
+				(font
+					(size 1.27 1.27)
+				)
+			)
+		)
 		(pin "4"
 		)
@@
 			)
 		)
-		(property "Footprint" ""
+		(property "Footprint" "Resistor_SMD:R_0603_1608Metric"
 			(at 149.352 97.79 90)
 			(hide yes)
@@
 			)
 		)
+		(property "LCSC Part" "C25804"
+			(at 151.13 97.79 0)
+			(hide yes)
+			(show_name no)
+			(do_not_autoplace no)
+			(effects
+				(font
+					(size 1.27 1.27)
+				)
+			)
+		)
 		(pin "1"
 		)
@@
 			)
 		)
-		(property "Value" "1u"
+		(property "Value" "1uF"
 			(at 219.71 100.3299 0)
 			(show_name no)
@@
 			)
 		)
-		(property "Footprint" ""
+		(property "Footprint" "Capacitor_SMD:C_0603_1608Metric"
 			(at 216.8652 102.87 0)
 			(hide yes)
@@
 			)
 		)
+		(property "LCSC Part" "C15849"
+			(at 215.9 99.06 0)
+			(hide yes)
+			(show_name no)
+			(do_not_autoplace no)
+			(effects
+				(font
+					(size 1.27 1.27)
+				)
+			)
+		)
 		(pin "1"
 		)
@@
 			)
 		)
-		(property "Value" "4.7u"
+		(property "Value" "4.7uF"
 			(at 72.39 100.3299 0)
 			(show_name no)
@@
 			)
 		)
-		(property "Footprint" ""
+		(property "Footprint" "Capacitor_SMD:C_0603_1608Metric"
 			(at 69.5452 102.87 0)
 			(hide yes)
@@
 			(at 68.58 99.06 0)
 			(hide yes)
+			(show_name no)
+			(do_not_autoplace no)
+			(effects
+				(font
+					(size 1.27 1.27)
+				)
+			)
+		)
+		(property "LCSC Part" "C19666"
+			(at 68.58 99.06 0)
+			(hide yes)

Commit message: Snapshot before 3D model path rework
Parts:
- D4: footprint Diode_SMD:D_SMA -> PlantMonitor_JLC:D_SMA
Changed lines of the file:
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@@
 			)
 		)
-		(property "Footprint" "Diode_SMD:D_SMA"
+		(property "Footprint" "PlantMonitor_JLC:D_SMA"
 			(at 220.345 76.2 0)
 			(hide yes)

Commit message: pre-order baseline
Other:
- company: (none) -> MuffinByteLabs
- title: (none) -> ESP32-S3 Plant Monitor
Changed lines of the file:
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@@
 	(generator_version "10.0")
 	(paper "A4")
+	(title_block
+		(title "ESP32-S3 Plant Monitor")
+		(date "2026-08-21")
+		(rev "A")
+		(company "MuffinByteLabs")
+		(comment 1 "Designed by Ray Malik")
+		(comment 2 "4-layer JLC04161H-7628, 1.6 mm, HASL lead-free, green mask")
+		(comment 3 "Fabrication and assembly: JLCPCB")
+	)
 	(junction
 		(at 139.7 67.31)
