File: hardware/08_Mechanical.kicad_sch (KiCad schematic)
At the start: 0 parts

Commit message: Pre-layout finalization and second design review pass (Rev A)
Parts:
- added H1, H2, H3, H4: MountingHole, MountingHole:MountingHole_3.2mm_M3, symbol Mechanical:MountingHole
- added TP1, TP2, TP3, TP4, TP5, TP6, TP7: TestPoint, TestPoint:TestPoint_Pad_D1.5mm, symbol Connector:TestPoint
- added TP8: TestPoint, TestPoint:TestPoint_THTPad_D2.0mm_Drill1.0mm, symbol Connector:TestPoint
Connections:
- new net +3V3: TP3.1
- new net +5V_PROT: TP1.1
- new net ADC_SOIL: TP6.1
- new net BAT_SENSE: TP5.1
- new net GND: TP7.1, TP8.1
- new net VBAT: TP4.1
- new net VSYS: TP2.1

Commit message: pre-order baseline
Other:
- company: (none) -> MuffinByteLabs
- title: (none) -> ESP32-S3 Plant Monitor
Changed lines of the file:
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@@
 	(generator_version "10.0")
 	(paper "A4")
+	(title_block
+		(title "ESP32-S3 Plant Monitor")
+		(date "2026-08-21")
+		(rev "A")
+		(company "MuffinByteLabs")
+		(comment 1 "Designed by Ray Malik")
+		(comment 2 "4-layer JLC04161H-7628, 1.6 mm, HASL lead-free, green mask")
+		(comment 3 "Fabrication and assembly: JLCPCB")
+	)
 	(wire
 		(pts
