File: hardware/ESP32S3_PlantMonitor.kicad_sch (KiCad schematic)
At the start: 0 parts

Commit message: pre-order baseline
Other:
- company: (none) -> MuffinByteLabs
- title: 01_System -> ESP32-S3 Plant Monitor
Changed lines of the file:
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@@
 	(paper "A4")
 	(title_block
-		(title "01_System")
-		(date "2026-07-03")
+		(title "ESP32-S3 Plant Monitor")
+		(date "2026-08-21")
 		(rev "A")
+		(company "MuffinByteLabs")
+		(comment 1 "Designed by Ray Malik")
+		(comment 2 "4-layer JLC04161H-7628, 1.6 mm, HASL lead-free, green mask")
+		(comment 3 "Fabrication and assembly: JLCPCB")
 	)
 	(sheet
